Commit message: xacro edits to match real robot and gazebo

File: src/ur3e_setup/urdf/ur_mrc_gazebo.xacro (robot description, xacro)
@@ -1,22 +1,5 @@
 <?xml version="1.0"?>
 <robot xmlns:xacro="http://wiki.ros.org/xacro" name="$(arg robot_model)_robot">
-  <!--
-    This is a top-level xacro instantiating the Gazebo-specific version of the
-    'ur_robot' macro (ie: 'ur_robot_gazebo') and passing it values for all its
-    required arguments.
-    This file should be considered the Gazebo-specific variant of the file
-    with the same name in the ur_description package. It accepts the same
-    arguments, but instead of configuring everything for a real robot, will
-    generate a Gazebo-compatible URDF with a ros_control hardware_interface
-    attached to it.
-    Only use this top-level xacro if you plan on spawning the robot in Gazebo
-    'by itself', without any gripper or any other geometry attached.
-    If you need to attach an end-effector, camera or need to integrate the
-    robot into a larger workcell and want to spawn that as a single entity in
-    Gazebo, DO NOT EDIT THIS FILE.
-    Instead: create a new top-level xacro, give it a proper name, include the
-    required '.xacro' files, instantiate the models (ie: call the macros) and
-    connect everything by adding the appropriate joints.
-  -->
+  <!--  This is a top-level xacro for UR3e arm stand in MRC RAL lab. -->
   <!--
     Import main macro.
@@ -73,30 +56,30 @@
     <origin xyz="0 0 0" rpy="0 0 0"/>
   </joint>
-<!-- Adding table surface to avoid collisions -->
-<link name="mount_table_link">
-    <visual>
-        <origin xyz="0 0 0" rpy="0 0 0"/>
-        <geometry>
-            <box size="1.12 0.805 0.766"/>
-        </geometry>
-        <material name="orange">
-            <color rgba="0.95 0.88 0.42 1.0"/>
-        </material>
-    </visual>
-    <collision>
-        <origin xyz="0 0 0" rpy="0 0 0"/>
-        <geometry>
-            <box size="1.12 0.805 0.766"/>
-        </geometry>
-    </collision>
-    <inertial>
-      <mass value="10.0" />
-      <inertia  ixx="1.0" ixy="0.0"  ixz="0.0"  iyy="1.0"  iyz="0.0"  izz="1.0" />
-    </inertial>
-</link>
-<joint name="mount_table_joint" type="fixed">
-    <parent link="world" />
-    <child link="mount_table_link" />
-    <origin xyz="0 0.3125 0.383" rpy="0 0 0" />
-</joint>
+  <!-- Adding table surface to avoid collisions -->
+  <link name="mount_table_link">
+      <visual>
+          <origin xyz="0 0 0" rpy="0 0 0"/>
+          <geometry>
+              <box size="1.12 0.805 0.766"/>
+          </geometry>
+          <material name="orange">
+              <color rgba="0.95 0.88 0.42 1.0"/>
+          </material>
+      </visual>
+      <collision>
+          <origin xyz="0 0 0" rpy="0 0 0"/>
+          <geometry>
+              <box size="1.12 0.805 0.766"/>
+          </geometry>
+      </collision>
+      <inertial>
+        <mass value="10.0" />
+        <inertia  ixx="1.0" ixy="0.0"  ixz="0.0"  iyy="1.0"  iyz="0.0"  izz="1.0" />
+      </inertial>
+  </link>
+  <joint name="mount_table_joint" type="fixed">
+      <parent link="world" />
+      <child link="mount_table_link" />
+      <origin xyz="0 0.3125 0.383" rpy="0 0 0" />
+  </joint>
 </robot>
